Commit message: improve building, streamline gripper config

File: mujoco/urdf/gripper_mujoco.urdf (robot description, URDF)
Before this commit: robot gripper, 42 links, 41 joints
Links:
- link finger_1_finger_hook_link: mass 0.00652777777778 -> 0.006444241316270568; geometry collision box size=0.0385 0.028 0.0009; visual box size=0.0385 0.028 0.0009
- link finger_1_segment_link_1: mass 0.00652777777778 -> 0.006444241316270568
- link finger_1_segment_link_10: mass 0.00652777777778 -> 0.006444241316270568
- link finger_1_segment_link_2: mass 0.00652777777778 -> 0.006444241316270568
- link finger_1_segment_link_3: mass 0.00652777777778 -> 0.006444241316270568
- link finger_1_segment_link_4: mass 0.00652777777778 -> 0.006444241316270568
- link finger_1_segment_link_5: mass 0.00652777777778 -> 0.006444241316270568
- link finger_1_segment_link_6: mass 0.00652777777778 -> 0.006444241316270568
- link finger_1_segment_link_7: mass 0.00652777777778 -> 0.006444241316270568
- link finger_1_segment_link_8: mass 0.00652777777778 -> 0.006444241316270568
- link finger_1_segment_link_9: mass 0.00652777777778 -> 0.006444241316270568
- link finger_2_finger_hook_link: mass 0.00652777777778 -> 0.006444241316270568; geometry collision box size=0.0385 0.028 0.0009; visual box size=0.0385 0.028 0.0009
- link finger_2_segment_link_1: mass 0.00652777777778 -> 0.006444241316270568
- link finger_2_segment_link_10: mass 0.00652777777778 -> 0.006444241316270568
- link finger_2_segment_link_2: mass 0.00652777777778 -> 0.006444241316270568
- link finger_2_segment_link_3: mass 0.00652777777778 -> 0.006444241316270568
- link finger_2_segment_link_4: mass 0.00652777777778 -> 0.006444241316270568
- link finger_2_segment_link_5: mass 0.00652777777778 -> 0.006444241316270568
- link finger_2_segment_link_6: mass 0.00652777777778 -> 0.006444241316270568
- link finger_2_segment_link_7: mass 0.00652777777778 -> 0.006444241316270568
- link finger_2_segment_link_8: mass 0.00652777777778 -> 0.006444241316270568
- link finger_2_segment_link_9: mass 0.00652777777778 -> 0.006444241316270568
- link finger_3_finger_hook_link: mass 0.00652777777778 -> 0.006444241316270568; geometry collision box size=0.0385 0.028 0.0009; visual box size=0.0385 0.028 0.0009
- link finger_3_segment_link_1: mass 0.00652777777778 -> 0.006444241316270568
- link finger_3_segment_link_10: mass 0.00652777777778 -> 0.006444241316270568
- link finger_3_segment_link_2: mass 0.00652777777778 -> 0.006444241316270568
- link finger_3_segment_link_3: mass 0.00652777777778 -> 0.006444241316270568
- link finger_3_segment_link_4: mass 0.00652777777778 -> 0.006444241316270568
- link finger_3_segment_link_5: mass 0.00652777777778 -> 0.006444241316270568
- link finger_3_segment_link_6: mass 0.00652777777778 -> 0.006444241316270568
- link finger_3_segment_link_7: mass 0.00652777777778 -> 0.006444241316270568
- link finger_3_segment_link_8: mass 0.00652777777778 -> 0.006444241316270568
- link finger_3_segment_link_9: mass 0.00652777777778 -> 0.006444241316270568
Joints:
- joint finger_1_finger_hook_joint: origin xyz=0.0235 0 0 rpy=0 -1.57079632679 0 -> xyz=0.0235 0 0 rpy=0 -1.5707963267948502 0
- joint finger_1_prismatic_joint: origin xyz=0.0                    0.0                    0 rpy=4.71238898038                    4.71238898038                    1.57079632679 -> xyz=0.0                    0.0                    0 rpy=4.71238898038469                    4.71238898038469                    1.5707963267948966
- joint finger_2_finger_hook_joint: origin xyz=0.0235 0 0 rpy=0 -1.57079632679 0 -> xyz=0.0235 0 0 rpy=0 -1.5707963267948502 0
- joint finger_2_prismatic_joint: origin xyz=0.0                    -0.0                    0 rpy=4.71238898038                    4.71238898038                    -0.523598775598 -> xyz=0.0                    -0.0                    0 rpy=4.71238898038469                    4.71238898038469                    -0.5235987755982987
- joint finger_3_finger_hook_joint: origin xyz=0.0235 0 0 rpy=0 -1.57079632679 0 -> xyz=0.0235 0 0 rpy=0 -1.5707963267948502 0
- joint finger_3_prismatic_joint: origin xyz=-0.0                    -0.0                    0 rpy=4.71238898038                    4.71238898038                    -2.61799387799 -> xyz=-0.0                    -0.0                    0 rpy=4.71238898038469                    4.71238898038469                    -2.617993877991494
- joint palm_prismatic_joint: origin xyz=0 0 0 rpy=0 -1.57079632679 0 -> xyz=0 0 0 rpy=0 -1.5707963267948966 0
- joint to_segmented_finger_1: origin xyz=0.129 -0.007 0 rpy=1.57079632679 0 0 -> xyz=0.129 -0.007 0 rpy=1.5707963267948966 0 0
- joint to_segmented_finger_2: origin xyz=0.129 -0.007 0 rpy=1.57079632679 0 0 -> xyz=0.129 -0.007 0 rpy=1.5707963267948966 0 0
- joint to_segmented_finger_3: origin xyz=0.129 -0.007 0 rpy=1.57079632679 0 0 -> xyz=0.129 -0.007 0 rpy=1.5707963267948966 0 0
- joint world_to_base: origin xyz=0 0 1 rpy=3.14159265359 0 0 -> xyz=0 0 1 rpy=3.141592653589793 0 0

File: mujoco/urdf/gripper_task.urdf (robot description, URDF)
Before this commit: robot gripper_task, 42 links, 41 joints
Links:
- link finger_1_finger_hook_link: mass 0.00652777777778 -> 0.006444241316270568; geometry collision box size=0.0385 0.028 0.0009; visual box size=0.0385 0.028 0.0009
- link finger_1_segment_link_1: mass 0.00652777777778 -> 0.006444241316270568
- link finger_1_segment_link_10: mass 0.00652777777778 -> 0.006444241316270568
- link finger_1_segment_link_2: mass 0.00652777777778 -> 0.006444241316270568
- link finger_1_segment_link_3: mass 0.00652777777778 -> 0.006444241316270568
- link finger_1_segment_link_4: mass 0.00652777777778 -> 0.006444241316270568
- link finger_1_segment_link_5: mass 0.00652777777778 -> 0.006444241316270568
- link finger_1_segment_link_6: mass 0.00652777777778 -> 0.006444241316270568
- link finger_1_segment_link_7: mass 0.00652777777778 -> 0.006444241316270568
- link finger_1_segment_link_8: mass 0.00652777777778 -> 0.006444241316270568
- link finger_1_segment_link_9: mass 0.00652777777778 -> 0.006444241316270568
- link finger_2_finger_hook_link: mass 0.00652777777778 -> 0.006444241316270568; geometry collision box size=0.0385 0.028 0.0009; visual box size=0.0385 0.028 0.0009
- link finger_2_segment_link_1: mass 0.00652777777778 -> 0.006444241316270568
- link finger_2_segment_link_10: mass 0.00652777777778 -> 0.006444241316270568
- link finger_2_segment_link_2: mass 0.00652777777778 -> 0.006444241316270568
- link finger_2_segment_link_3: mass 0.00652777777778 -> 0.006444241316270568
- link finger_2_segment_link_4: mass 0.00652777777778 -> 0.006444241316270568
- link finger_2_segment_link_5: mass 0.00652777777778 -> 0.006444241316270568
- link finger_2_segment_link_6: mass 0.00652777777778 -> 0.006444241316270568
- link finger_2_segment_link_7: mass 0.00652777777778 -> 0.006444241316270568
- link finger_2_segment_link_8: mass 0.00652777777778 -> 0.006444241316270568
- link finger_2_segment_link_9: mass 0.00652777777778 -> 0.006444241316270568
- link finger_3_finger_hook_link: mass 0.00652777777778 -> 0.006444241316270568; geometry collision box size=0.0385 0.028 0.0009; visual box size=0.0385 0.028 0.0009
- link finger_3_segment_link_1: mass 0.00652777777778 -> 0.006444241316270568
- link finger_3_segment_link_10: mass 0.00652777777778 -> 0.006444241316270568
- link finger_3_segment_link_2: mass 0.00652777777778 -> 0.006444241316270568
- link finger_3_segment_link_3: mass 0.00652777777778 -> 0.006444241316270568
- link finger_3_segment_link_4: mass 0.00652777777778 -> 0.006444241316270568
- link finger_3_segment_link_5: mass 0.00652777777778 -> 0.006444241316270568
- link finger_3_segment_link_6: mass 0.00652777777778 -> 0.006444241316270568
- link finger_3_segment_link_7: mass 0.00652777777778 -> 0.006444241316270568
- link finger_3_segment_link_8: mass 0.00652777777778 -> 0.006444241316270568
- link finger_3_segment_link_9: mass 0.00652777777778 -> 0.006444241316270568
Joints:
- joint finger_1_finger_hook_joint: origin xyz=0.0235 0 0 rpy=0 -1.57079632679 0 -> xyz=0.0235 0 0 rpy=0 -1.5707963267948502 0
- joint finger_1_prismatic_joint: origin xyz=0.0                    0.0                    0 rpy=4.71238898038                    4.71238898038                    1.57079632679 -> xyz=0.0                    0.0                    0 rpy=4.71238898038469                    4.71238898038469                    1.5707963267948966
- joint finger_2_finger_hook_joint: origin xyz=0.0235 0 0 rpy=0 -1.57079632679 0 -> xyz=0.0235 0 0 rpy=0 -1.5707963267948502 0
- joint finger_2_prismatic_joint: origin xyz=0.0                    -0.0                    0 rpy=4.71238898038                    4.71238898038                    -0.523598775598 -> xyz=0.0                    -0.0                    0 rpy=4.71238898038469                    4.71238898038469                    -0.5235987755982987
- joint finger_3_finger_hook_joint: origin xyz=0.0235 0 0 rpy=0 -1.57079632679 0 -> xyz=0.0235 0 0 rpy=0 -1.5707963267948502 0
- joint finger_3_prismatic_joint: origin xyz=-0.0                    -0.0                    0 rpy=4.71238898038                    4.71238898038                    -2.61799387799 -> xyz=-0.0                    -0.0                    0 rpy=4.71238898038469                    4.71238898038469                    -2.617993877991494
- joint palm_prismatic_joint: origin xyz=0 0 0 rpy=0 -1.57079632679 0 -> xyz=0 0 0 rpy=0 -1.5707963267948966 0
- joint to_segmented_finger_1: origin xyz=0.129 -0.007 0 rpy=1.57079632679 0 0 -> xyz=0.129 -0.007 0 rpy=1.5707963267948966 0 0
- joint to_segmented_finger_2: origin xyz=0.129 -0.007 0 rpy=1.57079632679 0 0 -> xyz=0.129 -0.007 0 rpy=1.5707963267948966 0 0
- joint to_segmented_finger_3: origin xyz=0.129 -0.007 0 rpy=1.57079632679 0 0 -> xyz=0.129 -0.007 0 rpy=1.5707963267948966 0 0
- joint world_to_base: origin xyz=0 0 0.335 rpy=3.14159265359 0 0 -> xyz=0 0 0.386 rpy=3.141592653589793 0 0

File: mujoco/urdf/panda_and_gripper_mujoco.urdf (robot description, URDF)
Before this commit: robot panda_and_gripper, 51 links, 50 joints
Links:
- link finger_1_finger_hook_link: mass 0.00652777777778 -> 0.006444241316270568; geometry collision box size=0.0385 0.028 0.0009; visual box size=0.0385 0.028 0.0009
- link finger_1_segment_link_1: mass 0.00652777777778 -> 0.006444241316270568
- link finger_1_segment_link_10: mass 0.00652777777778 -> 0.006444241316270568
- link finger_1_segment_link_2: mass 0.00652777777778 -> 0.006444241316270568
- link finger_1_segment_link_3: mass 0.00652777777778 -> 0.006444241316270568
- link finger_1_segment_link_4: mass 0.00652777777778 -> 0.006444241316270568
- link finger_1_segment_link_5: mass 0.00652777777778 -> 0.006444241316270568
- link finger_1_segment_link_6: mass 0.00652777777778 -> 0.006444241316270568
- link finger_1_segment_link_7: mass 0.00652777777778 -> 0.006444241316270568
- link finger_1_segment_link_8: mass 0.00652777777778 -> 0.006444241316270568
- link finger_1_segment_link_9: mass 0.00652777777778 -> 0.006444241316270568
- link finger_2_finger_hook_link: mass 0.00652777777778 -> 0.006444241316270568; geometry collision box size=0.0385 0.028 0.0009; visual box size=0.0385 0.028 0.0009
- link finger_2_segment_link_1: mass 0.00652777777778 -> 0.006444241316270568
- link finger_2_segment_link_10: mass 0.00652777777778 -> 0.006444241316270568
- link finger_2_segment_link_2: mass 0.00652777777778 -> 0.006444241316270568
- link finger_2_segment_link_3: mass 0.00652777777778 -> 0.006444241316270568
- link finger_2_segment_link_4: mass 0.00652777777778 -> 0.006444241316270568
- link finger_2_segment_link_5: mass 0.00652777777778 -> 0.006444241316270568
- link finger_2_segment_link_6: mass 0.00652777777778 -> 0.006444241316270568
- link finger_2_segment_link_7: mass 0.00652777777778 -> 0.006444241316270568
- link finger_2_segment_link_8: mass 0.00652777777778 -> 0.006444241316270568
- link finger_2_segment_link_9: mass 0.00652777777778 -> 0.006444241316270568
- link finger_3_finger_hook_link: mass 0.00652777777778 -> 0.006444241316270568; geometry collision box size=0.0385 0.028 0.0009; visual box size=0.0385 0.028 0.0009
- link finger_3_segment_link_1: mass 0.00652777777778 -> 0.006444241316270568
- link finger_3_segment_link_10: mass 0.00652777777778 -> 0.006444241316270568
- link finger_3_segment_link_2: mass 0.00652777777778 -> 0.006444241316270568
- link finger_3_segment_link_3: mass 0.00652777777778 -> 0.006444241316270568
- link finger_3_segment_link_4: mass 0.00652777777778 -> 0.006444241316270568
- link finger_3_segment_link_5: mass 0.00652777777778 -> 0.006444241316270568
- link finger_3_segment_link_6: mass 0.00652777777778 -> 0.006444241316270568
- link finger_3_segment_link_7: mass 0.00652777777778 -> 0.006444241316270568
- link finger_3_segment_link_8: mass 0.00652777777778 -> 0.006444241316270568
- link finger_3_segment_link_9: mass 0.00652777777778 -> 0.006444241316270568
Joints:
- joint finger_1_finger_hook_joint: origin xyz=0.0235 0 0 rpy=0 -1.57079632679 0 -> xyz=0.0235 0 0 rpy=0 -1.5707963267948502 0
- joint finger_1_prismatic_joint: origin xyz=0.0                    0.0                    0 rpy=4.71238898038                    4.71238898038                    1.57079632679 -> xyz=0.0                    0.0                    0 rpy=4.71238898038469                    4.71238898038469                    1.5707963267948966
- joint finger_2_finger_hook_joint: origin xyz=0.0235 0 0 rpy=0 -1.57079632679 0 -> xyz=0.0235 0 0 rpy=0 -1.5707963267948502 0
- joint finger_2_prismatic_joint: origin xyz=0.0                    -0.0                    0 rpy=4.71238898038                    4.71238898038                    -0.523598775598 -> xyz=0.0                    -0.0                    0 rpy=4.71238898038469                    4.71238898038469                    -0.5235987755982987
- joint finger_3_finger_hook_joint: origin xyz=0.0235 0 0 rpy=0 -1.57079632679 0 -> xyz=0.0235 0 0 rpy=0 -1.5707963267948502 0
- joint finger_3_prismatic_joint: origin xyz=-0.0                    -0.0                    0 rpy=4.71238898038                    4.71238898038                    -2.61799387799 -> xyz=-0.0                    -0.0                    0 rpy=4.71238898038469                    4.71238898038469                    -2.617993877991494
- joint palm_prismatic_joint: origin xyz=0 0 0 rpy=0 -1.57079632679 0 -> xyz=0 0 0 rpy=0 -1.5707963267948966 0
- joint panda_joint2: origin xyz=0 0 0 rpy=-1.57079632679 0 0 -> xyz=0 0 0 rpy=-1.5707963267948966 0 0
- joint panda_joint3: origin xyz=0 -0.316 0 rpy=1.57079632679 0 0 -> xyz=0 -0.316 0 rpy=1.5707963267948966 0 0
- joint panda_joint4: origin xyz=0.0825 0 0 rpy=1.57079632679 0 0 -> xyz=0.0825 0 0 rpy=1.5707963267948966 0 0
- joint panda_joint5: origin xyz=-0.0825 0.384 0 rpy=-1.57079632679 0 0 -> xyz=-0.0825 0.384 0 rpy=-1.5707963267948966 0 0
- joint panda_joint6: origin xyz=0 0 0 rpy=1.57079632679 0 0 -> xyz=0 0 0 rpy=1.5707963267948966 0 0
- joint panda_joint7: origin xyz=0.088 0 0 rpy=1.57079632679 0 0 -> xyz=0.088 0 0 rpy=1.5707963267948966 0 0
- joint panda_to_eef_base_joint: origin xyz=0 0 0.25 rpy=0 0 -0.785398163397 -> xyz=0 0 0.25 rpy=0 0 -0.7853981633974483
- joint to_segmented_finger_1: origin xyz=0.129 -0.007 0 rpy=1.57079632679 0 0 -> xyz=0.129 -0.007 0 rpy=1.5707963267948966 0 0
- joint to_segmented_finger_2: origin xyz=0.129 -0.007 0 rpy=1.57079632679 0 0 -> xyz=0.129 -0.007 0 rpy=1.5707963267948966 0 0
- joint to_segmented_finger_3: origin xyz=0.129 -0.007 0 rpy=1.57079632679 0 0 -> xyz=0.129 -0.007 0 rpy=1.5707963267948966 0 0

File: mujoco/urdf/panda_mujoco.urdf (robot description, URDF)
Before this commit: robot panda, 10 links, 9 joints
Joints:
- joint panda_joint2: origin xyz=0 0 0 rpy=-1.57079632679 0 0 -> xyz=0 0 0 rpy=-1.5707963267948966 0 0
- joint panda_joint3: origin xyz=0 -0.316 0 rpy=1.57079632679 0 0 -> xyz=0 -0.316 0 rpy=1.5707963267948966 0 0
- joint panda_joint4: origin xyz=0.0825 0 0 rpy=1.57079632679 0 0 -> xyz=0.0825 0 0 rpy=1.5707963267948966 0 0
- joint panda_joint5: origin xyz=-0.0825 0.384 0 rpy=-1.57079632679 0 0 -> xyz=-0.0825 0.384 0 rpy=-1.5707963267948966 0 0
- joint panda_joint6: origin xyz=0 0 0 rpy=1.57079632679 0 0 -> xyz=0 0 0 rpy=1.5707963267948966 0 0
- joint panda_joint7: origin xyz=0.088 0 0 rpy=1.57079632679 0 0 -> xyz=0.088 0 0 rpy=1.5707963267948966 0 0

File: mujoco/xacro/gripper_task.urdf.xacro (robot description, xacro)
@@ -9,15 +9,22 @@
 	<xacro:include filename="${path_to_top}/xacro/gripper.xacro"/>
 	<xacro:add_gripper path_to_top="${path_to_top}"/>
-  <!-- attach gripper to the ground for gazebo -->
+	<!-- height for fingertips to just not touch the ground, then height to raise
+	past that. Note that this height is calibrated manually using mujoco and with
+  checking the wrist z sensor for contact. This is calibrated AFTER the gripper
+	has settled (ie joint controller stiffness accounted for)-->
+	<xacro:property name="fingertip_touches_ground" value="0.376"/>
+	<xacro:property name="fingertip_clearance" value="0.01"/>
+	<xacro:property name="h" value="${fingertip_touches_ground + fingertip_clearance}"/>
+  <!-- attach gripper to the ground for mujoco -->
 	<link name="world"/>
 	<joint name="world_to_base" type="prismatic">
-		<origin xyz="0 0 0.335" rpy="${pi} 0 0"/> <!-- 0.325 is fingertips just not touching-->
+		<origin xyz="0 0 ${h}" rpy="${pi} 0 0"/>
 		<axis xyz="0 0 1" rpy="0 0 0"/>
 		<parent link="world"/>
 		<child link="gripper_base_link"/>
 		<limit effort="1e3"
-        			 lower="-1"
-        			 upper="1"
-        			 velocity="1"/>
+					 lower="-1"
+					 upper="1"
+					 velocity="1"/>
     <dynamics damping="1"/>
 	</joint>

File: xacro/gripper.main.xacro (robot description, xacro)
@@ -1,25 +1,17 @@
 <?xml version="1.0"?>
 <robot xmlns:xacro="http://ros.org/wiki/xacro">
-  <xacro:macro name="gripper" params="is_segmented">
-  	<!-- retrieve info about the gripper
-    <xacro:property name="filename" value="$(find gripper_description)/config/gripper.yaml"/>
-    <xacro:property name="dictionary" value="${xacro.load_yaml(filename)}"/>
-    <xacro:property name="is_segmented" value="${dictionary['gripper_config']['is_segmented']}"/>
-    -->
-    <xacro:property name="filename" value="../config/gripper.yaml"/>
-    <xacro:property name="dictionary" value="${xacro.load_yaml(filename)}"/>
-    <xacro:property name="finger_displacement_min" value="${dictionary['params']['xy_min']}"/>
-    <xacro:property name="finger_displacement_max" value="${dictionary['params']['xy_max']}"/>
-    <xacro:property name="palm_displacement_min" value="${dictionary['params']['z_min']}"/>
-    <xacro:property name="palm_displacement_max" value="${dictionary['params']['z_max']}"/>
-    <!-- <xacro:property name="is_segmented" value="${dictionary['gripper_config']['is_segmented']}"/> -->
+  <xacro:macro name="gripper" params="yaml_dict">
+		<!-- load the gripper config information -->
+    <xacro:property name="filename" value="${path_to_top}/config/gripper.yaml"/>
+    <xacro:property name="yaml_dict" value="${xacro.load_yaml(filename)}"/>
+    <!-- extract the gripper config information -->
+    <xacro:property name="is_segmented" value="${yaml_dict['gripper_config']['is_segmented']}"/>
+    <xacro:property name="finger_displacement_min" value="${yaml_dict['gripper_params']['xy_min']}"/>
+    <xacro:property name="finger_displacement_max" value="${yaml_dict['gripper_params']['xy_max']}"/>
+    <xacro:property name="palm_displacement_min" value="${yaml_dict['gripper_params']['z_min']}"/>
+    <xacro:property name="palm_displacement_max" value="${yaml_dict['gripper_params']['z_max']}"/>
+    <xacro:property name="finger_angle_min" value="${-1 * yaml_dict['gripper_params']['angle_max_abs']}"/>
+    <xacro:property name="finger_angle_max" value="${yaml_dict['gripper_params']['angle_max_abs']}"/>
   	<!-- PARAMETERS TO BE SET BY HAND -->
-    <!-- Define motion limits of each joint, these all in SI units -->
-    <xacro:property name="finger_displacement_min" value="0.049"/> <!-- based on 32 revs home to max -->
-    <xacro:property name="finger_displacement_max" value="0.134"/> <!-- set in Gripper_v2.h (Arduino library)-->
-    <xacro:property name="finger_angle_min" value="-0.7"/>
-    <xacro:property name="finger_angle_max" value="0.7"/>
-    <xacro:property name="palm_displacement_min" value="0.0"/> <!-- set in Gripper_v2.h (Arduino library)-->
-    <xacro:property name="palm_displacement_max" value="0.165"/> <!-- based on 34 revs home to max-->
     <!-- Define limits of each joint, these all in SI units -->
     <xacro:property name="finger_displacement_velocity" value="0.015"/>
@@ -93,5 +85,4 @@
     <!-- BASE LINK -->
     <link name="gripper_base_link">
-      <!-- <xacro:default_inertial mass="1.0"/> -->
       <xacro:set_inertia key="1"/>
       <visual>
@@ -123,5 +114,4 @@
       <!-- Intermediate link for prismatic joint -->
       <link name="finger_${number}_intermediate">
-        <!-- <xacro:default_inertial mass="0.03"/> -->
         <xacro:set_inertia key="2"/>
         <visual>
@@ -140,5 +130,4 @@
         <!-- If we are using rigid fingers -->
         <xacro:if value="${not is_segmented}">
-          <!-- <xacro:default_inertial mass="0.3"/> -->
           <xacro:set_inertia key="4"/>
           <visual>
@@ -155,5 +144,4 @@
         <!-- If we are using segmented fingers -->
         <xacro:if value="${is_segmented}">
-          <!-- <xacro:default_inertial mass="0.3"/> -->
           <xacro:set_inertia key="3"/>
           <visual>
@@ -200,5 +188,4 @@
     <!-- PALM -->
     <link name="palm">
-      <!-- <xacro:default_inertial mass="0.05" /> -->
       <xacro:set_inertia key="5"/>
       <visual>
