Commit message: improve building, streamline gripper config

File: xacro/gripper.segmented_fingers.xacro (robot description, xacro)
@@ -1,13 +1,16 @@
 <?xml version="1.0"?>
 <robot xmlns:xacro="http://ros.org/wiki/xacro">
-  <xacro:macro name="segmented_finger" params="prefix num_segments torsion">
+  <xacro:macro name="segmented_finger" params="prefix yaml_dict">
+    <!-- extract the gripper config information -->
+    <xacro:property name="is_segmented" value="${yaml_dict['gripper_config']['is_segmented']}"/>
+    <xacro:property name="num_segments" value="${yaml_dict['gripper_config']['num_segments']}"/>
+    <xacro:property name="torsion" value="${yaml_dict['gripper_config']['torsion']}"/>
+    <xacro:property name="finger_length" value="${yaml_dict['gripper_params']['finger_length']}"/>
+    <xacro:property name="finger_width" value="${yaml_dict['gripper_params']['finger_width']}"/>
+    <xacro:property name="finger_thickness" value="${yaml_dict['gripper_params']['finger_thickness']}"/>
+    <xacro:property name="finger_mass" value="${yaml_dict['gripper_params']['finger_mass']}"/>
+    <xacro:property name="hook_length" value="${yaml_dict['gripper_params']['hook_length']}"/>
+    <xacro:property name="hook_angle" value="${yaml_dict['gripper_params']['hook_angle_degrees'] * (3.1415926535897 / 180.0)}"/>
   	<!-- PARAMETERS TO BE SET BY HAND -->
-    <!-- User defined variables -->
-    <xacro:property name="finger_length_mm" value="235.0"/>
-    <xacro:property name="hook_length_mm" value="35.0"/>
-    <xacro:property name="finger_width_mm" value="28.0"/>
-    <xacro:property name="finger_thickness_mm" value="0.9"/>
-    <xacro:property name="hook_angle_d" value="90.0"/>
-    <xacro:property name="finger_mass_g" value="75.0"/>
     <!-- macros to set the sdf elements, all here together for convienience -->
     <!-- Tags for gazebo, see: http://gazebosim.org/tutorials?tut=ros_urdf -->
@@ -37,12 +40,8 @@
     <!-- END OF PARAMETERS TO BE SET BY HAND -->
     <!-- Automatially calculated variables -->
-    <xacro:property name="finger_length" value="${finger_length_mm * 0.001}"/>
-    <xacro:property name="segment_length" value="${(finger_length_mm / num_segments) * 0.001}"/>
-    <xacro:property name="segment_width" value="${finger_width_mm * 0.001}"/>
-    <xacro:property name="segment_thickness" value="${finger_thickness_mm * 0.001}"/>
-    <xacro:property name="hook_length" value="${hook_length_mm * 0.001}"/>
-    <xacro:property name="hook_angle" value="${(hook_angle_d / 180.0) * 3.1415926535897}"/>
+    <xacro:property name="segment_length" value="${finger_length / float(num_segments)}"/>
+    <xacro:property name="segment_width" value="${finger_width}"/>
+    <xacro:property name="segment_thickness" value="${finger_thickness}"/>
     <!-- find inertia of each segment -->
-    <xacro:property name="finger_mass" value="${finger_mass_g * 0.001}"/>
     <xacro:property name="segment_mass"
       value="${(finger_mass * segment_length) / (finger_length + hook_length)}"/>
@@ -67,8 +66,4 @@
                  izz="${segment_izz * stability_factor}"
                 ixy="0.00" iyz="0.00" ixz="0.00" />
-        <!-- <inertia ixx="${1e-6 * stability_factor}"
-                 iyy="${1e-6 * stability_factor}"
-                 izz="${1e-6 * stability_factor}"
-                ixy="0.00" iyz="0.00" ixz="0.00" /> -->
       </inertial>
     </xacro:macro>
@@ -76,5 +71,5 @@
     <xacro:macro name="add_segment_link" params="number">
       <link name="${prefix}_segment_link_${number}">
-        <xacro:segment_inertial mass="${(75 * 0.001) / num_segments}" num="${number}"/>
+        <xacro:segment_inertial mass="${segment_mass / num_segments}" num="${number}"/>
         <visual>
           <origin xyz="${segment_length / 2} 0 0"
@@ -167,5 +162,5 @@
     <!-- Add the finger hook link -->
     <link name="${prefix}_finger_hook_link">
-      <xacro:segment_inertial mass="${(75 * 0.001) / num_segments}" num="${num_segments}"/>
+      <xacro:segment_inertial mass="${(finger_mass * 0.001) / num_segments}" num="${num_segments}"/>
       <visual>
         <origin xyz="${hook_length / 2} 0 0"

File: xacro/gripper.xacro (robot description, xacro)
@@ -14,19 +14,14 @@
 		<xacro:include filename="${path_to_top}/xacro/gripper.segmented_fingers.xacro"/>
 		<!-- load information from the gripper yaml file -->
-		<xacro:property name="dictionary" value="${xacro.load_yaml(filename)}"/>
-		<xacro:property name="is_segmented" value="${dictionary['gripper_config']['is_segmented']}"/>
-		<xacro:property name="num_segments" value="${dictionary['gripper_config']['num_segments']}"/>
-		<xacro:property name="torsion" value="${dictionary['gripper_config']['torsion']}"/>
-		<!-- create instances of gripper -->
-		<xacro:gripper is_segmented="${is_segmented}"/>
+		<xacro:property name="yaml_dict" value="${xacro.load_yaml(filename)}"/>
+		<xacro:property name="is_segmented" value="${yaml_dict['gripper_config']['is_segmented']}"/>
+		<!-- create instance of gripper -->
+		<xacro:gripper yaml_dict="${yaml_dict}"/>
 		<!-- macro for adding the segmented fingers onto the gripper-->
-		<xacro:macro name="add_fingers" params="segments">
+		<xacro:macro name="add_fingers">
 		  <!-- Create the fingers themselves -->
-		  <xacro:segmented_finger prefix="finger_1" num_segments="${segments}"
-		    torsion="${torsion}"/>
-		  <xacro:segmented_finger prefix="finger_2" num_segments="${segments}"
-		    torsion="${torsion}"/>
-		  <xacro:segmented_finger prefix="finger_3" num_segments="${segments}"
-		    torsion="${torsion}"/>
+		  <xacro:segmented_finger prefix="finger_1" yaml_dict="${yaml_dict}"/>
+		  <xacro:segmented_finger prefix="finger_2" yaml_dict="${yaml_dict}"/>
+		  <xacro:segmented_finger prefix="finger_3" yaml_dict="${yaml_dict}"/>
 		  <!-- adds the finger controller plugin to gazebo -->
 		  <xacro:gazebo_plugin/>
@@ -50,5 +45,5 @@
 		<!-- add the segmented fingers only if indicated in gripper.config -->
 		<xacro:if value="${is_segmented}">
-		  <xacro:add_fingers segments="${num_segments}"/>
+		  <xacro:add_fingers/>
 		</xacro:if>
   </xacro:macro>

Commit message: add free first joint option

File: mujoco/urdf/gripper_mujoco.urdf (robot description, URDF)
Before this commit: robot gripper, 42 links, 41 joints
Joints:
- removed joint to_segmented_finger_1
- removed joint to_segmented_finger_2
- removed joint to_segmented_finger_3
- added joint finger_1_segment_joint_0: type revolute, parent finger_1, child finger_1_segment_link_1, origin xyz=0.129 -0.007 0 rpy=1.5707963267948966 0 0, axis 0 1 0, limit lower=-1.0 upper=1.0 effort=1000.0 velocity=1.0
- added joint finger_2_segment_joint_0: type revolute, parent finger_2, child finger_2_segment_link_1, origin xyz=0.129 -0.007 0 rpy=1.5707963267948966 0 0, axis 0 1 0, limit lower=-1.0 upper=1.0 effort=1000.0 velocity=1.0
- added joint finger_3_segment_joint_0: type revolute, parent finger_3, child finger_3_segment_link_1, origin xyz=0.129 -0.007 0 rpy=1.5707963267948966 0 0, axis 0 1 0, limit lower=-1.0 upper=1.0 effort=1000.0 velocity=1.0

File: mujoco/urdf/gripper_task.urdf (robot description, URDF)
Before this commit: robot gripper_task, 42 links, 41 joints
Joints:
- removed joint to_segmented_finger_1
- removed joint to_segmented_finger_2
- removed joint to_segmented_finger_3
- added joint finger_1_segment_joint_0: type revolute, parent finger_1, child finger_1_segment_link_1, origin xyz=0.129 -0.007 0 rpy=1.5707963267948966 0 0, axis 0 1 0, limit lower=-1.0 upper=1.0 effort=1000.0 velocity=1.0
- added joint finger_2_segment_joint_0: type revolute, parent finger_2, child finger_2_segment_link_1, origin xyz=0.129 -0.007 0 rpy=1.5707963267948966 0 0, axis 0 1 0, limit lower=-1.0 upper=1.0 effort=1000.0 velocity=1.0
- added joint finger_3_segment_joint_0: type revolute, parent finger_3, child finger_3_segment_link_1, origin xyz=0.129 -0.007 0 rpy=1.5707963267948966 0 0, axis 0 1 0, limit lower=-1.0 upper=1.0 effort=1000.0 velocity=1.0

File: mujoco/urdf/panda_and_gripper_mujoco.urdf (robot description, URDF)
Before this commit: robot panda_and_gripper, 51 links, 50 joints
Joints:
- removed joint to_segmented_finger_1
- removed joint to_segmented_finger_2
- removed joint to_segmented_finger_3
- added joint finger_1_segment_joint_0: type revolute, parent finger_1, child finger_1_segment_link_1, origin xyz=0.129 -0.007 0 rpy=1.5707963267948966 0 0, axis 0 1 0, limit lower=-1.0 upper=1.0 effort=1000.0 velocity=1.0
- added joint finger_2_segment_joint_0: type revolute, parent finger_2, child finger_2_segment_link_1, origin xyz=0.129 -0.007 0 rpy=1.5707963267948966 0 0, axis 0 1 0, limit lower=-1.0 upper=1.0 effort=1000.0 velocity=1.0
- added joint finger_3_segment_joint_0: type revolute, parent finger_3, child finger_3_segment_link_1, origin xyz=0.129 -0.007 0 rpy=1.5707963267948966 0 0, axis 0 1 0, limit lower=-1.0 upper=1.0 effort=1000.0 velocity=1.0

File: urdf/gripper.urdf (robot description, URDF)
Before this commit: robot gripper, 42 links, 41 joints
Joints:
- removed joint to_segmented_finger_1
- removed joint to_segmented_finger_2
- removed joint to_segmented_finger_3
- added joint finger_1_segment_joint_0: type revolute, parent finger_1, child finger_1_segment_link_1, origin xyz=0.129 -0.007 0 rpy=1.5707963267948966 0 0, axis 0 1 0, limit lower=-1.0 upper=1.0 effort=1000.0 velocity=1.0
- added joint finger_2_segment_joint_0: type revolute, parent finger_2, child finger_2_segment_link_1, origin xyz=0.129 -0.007 0 rpy=1.5707963267948966 0 0, axis 0 1 0, limit lower=-1.0 upper=1.0 effort=1000.0 velocity=1.0
- added joint finger_3_segment_joint_0: type revolute, parent finger_3, child finger_3_segment_link_1, origin xyz=0.129 -0.007 0 rpy=1.5707963267948966 0 0, axis 0 1 0, limit lower=-1.0 upper=1.0 effort=1000.0 velocity=1.0

File: urdf/panda_and_gripper.urdf (robot description, URDF)
Before this commit: robot panda_and_gripper, 51 links, 50 joints
Joints:
- removed joint to_segmented_finger_1
- removed joint to_segmented_finger_2
- removed joint to_segmented_finger_3
- added joint finger_1_segment_joint_0: type revolute, parent finger_1, child finger_1_segment_link_1, origin xyz=0.129 -0.007 0 rpy=1.5707963267948966 0 0, axis 0 1 0, limit lower=-1.0 upper=1.0 effort=1000.0 velocity=1.0
- added joint finger_2_segment_joint_0: type revolute, parent finger_2, child finger_2_segment_link_1, origin xyz=0.129 -0.007 0 rpy=1.5707963267948966 0 0, axis 0 1 0, limit lower=-1.0 upper=1.0 effort=1000.0 velocity=1.0
- added joint finger_3_segment_joint_0: type revolute, parent finger_3, child finger_3_segment_link_1, origin xyz=0.129 -0.007 0 rpy=1.5707963267948966 0 0, axis 0 1 0, limit lower=-1.0 upper=1.0 effort=1000.0 velocity=1.0

File: xacro/gripper.segmented_fingers.xacro (robot description, xacro)
@@ -1,8 +1,9 @@
 <?xml version="1.0"?>
 <robot xmlns:xacro="http://ros.org/wiki/xacro">
-  <xacro:macro name="segmented_finger" params="prefix yaml_dict">
+  <xacro:macro name="segmented_finger" params="prefix yaml_dict connect_to x y z">
     <!-- extract the gripper config information -->
     <xacro:property name="is_segmented" value="${yaml_dict['gripper_config']['is_segmented']}"/>
     <xacro:property name="num_segments" value="${yaml_dict['gripper_config']['num_segments']}"/>
+    <xacro:property name="fixed_first_segment" value="${yaml_dict['gripper_config']['fixed_first_segment']}"/>
     <xacro:property name="torsion" value="${yaml_dict['gripper_config']['torsion']}"/>
     <xacro:property name="finger_length" value="${yaml_dict['gripper_params']['finger_length']}"/>
@@ -65,5 +66,5 @@
                  iyy="${segment_iyy * stability_factor}"
                  izz="${segment_izz * stability_factor}"
-                ixy="0.00" iyz="0.00" ixz="0.00" />
+                 ixy="0.00" iyz="0.00" ixz="0.00" />
       </inertial>
     </xacro:macro>
@@ -145,4 +146,26 @@
       </transmission>
     </xacro:macro>
+    <!-- TESTING: add a base joint connection -->
+    <xacro:if value="${fixed_first_segment}">
+    	<joint name="${prefix}_fixed_segment_connection" type="fixed">
+    		<origin xyz="${x_fix} ${y_fix} ${z_fix}" rpy="${pi/2} 0 0"/>
+		  	<parent link="${connect_to}"/>
+		  	<child link="${prefix}_segment_link_1"/>
+		  </joint>
+    </xacro:if>
+    <xacro:if value="${not fixed_first_segment}">
+		  <joint name="${prefix}_segment_joint_0" type="revolute">
+		  	<origin xyz="${x_fix} ${y_fix} ${z_fix}" rpy="${pi/2} 0 0"/>
+		  	<parent link="${connect_to}"/>
+		  	<child link="${prefix}_segment_link_1"/>
+		  	<axis xyz="0 1 0" rpy="0 0 0"/>
+		    <limit effort="1000.0"
+		          lower="-1.0"
+		          upper="1.0"
+		          velocity="1.0"/>
+		    <dynamics damping="${joint_damping}" friction="${joint_friction}"/>
+		  </joint>
+    </xacro:if>
+    <!-- END TESTING OF BASE JOINT (rather than fixed) -->
     <!-- Create the base link -->
     <xacro:add_segment_link number="1"/>

File: xacro/gripper.xacro (robot description, xacro)
@@ -21,12 +21,16 @@
 		<xacro:macro name="add_fingers">
 		  <!-- Create the fingers themselves -->
-		  <xacro:segmented_finger prefix="finger_1" yaml_dict="${yaml_dict}"/>
-		  <xacro:segmented_finger prefix="finger_2" yaml_dict="${yaml_dict}"/>
-		  <xacro:segmented_finger prefix="finger_3" yaml_dict="${yaml_dict}"/>
+		  <xacro:segmented_finger prefix="finger_1" yaml_dict="${yaml_dict}"
+		  												connect_to="finger_1" x="${x_fix}" y="${y_fix}" z="${z_fix}"/>
+		  <xacro:segmented_finger prefix="finger_2" yaml_dict="${yaml_dict}"
+		  												connect_to="finger_2" x="${x_fix}" y="${y_fix}" z="${z_fix}"/>
+		  <xacro:segmented_finger prefix="finger_3" yaml_dict="${yaml_dict}"
+		  												connect_to="finger_3" x="${x_fix}" y="${y_fix}" z="${z_fix}"/>
 		  <!-- adds the finger controller plugin to gazebo -->
 		  <xacro:gazebo_plugin/>
-		  <!-- attach them to the gripper -->
+		  <!-- OLD CODE: delete later if not needed
+			comment: attach them to the gripper
 		  <joint name="to_segmented_finger_1" type="fixed">
-		    <origin xyz="${x_fix} ${y_fix} ${z_fix}" rpy="${pi/2} 0 0"/>
+		    <origin xyz="${x_fix} ${y_fix} ${z_fix + 0.1}" rpy="${pi/2} 0 0"/>
 		    <parent link="finger_1"/>
 		    <child link="finger_1_segment_link_1"/>
@@ -42,4 +46,5 @@
 		    <child link="finger_3_segment_link_1"/>
 		  </joint>
+		  -->
 		</xacro:macro>
 		<!-- add the segmented fingers only if indicated in gripper.config -->
