Commit message: add seperate files for keyframes

File: mujoco/urdf/gripper_mujoco.urdf (robot description, URDF)
Before this commit: robot gripper, 42 links, 41 joints
Links:
- removed link finger_1_segment_link_10
- removed link finger_1_segment_link_7
- removed link finger_1_segment_link_8
- removed link finger_1_segment_link_9
- removed link finger_2_segment_link_10
- removed link finger_2_segment_link_7
- removed link finger_2_segment_link_8
- removed link finger_2_segment_link_9
- removed link finger_3_segment_link_10
- removed link finger_3_segment_link_7
- removed link finger_3_segment_link_8
- removed link finger_3_segment_link_9
- link finger_1_finger_hook_link: mass 0.006444241316270568 -> 0.010740402193784278
- link finger_1_segment_link_1: mass 0.006444241316270568 -> 0.010740402193784278; geometry collision box size=0.03916666666666666 0.028 0.0009; visual box size=0.03916666666666666 0.028 0.0009
- link finger_1_segment_link_2: mass 0.006444241316270568 -> 0.010740402193784278; geometry collision box size=0.03916666666666666 0.028 0.0009; visual box size=0.03916666666666666 0.028 0.0009
- link finger_1_segment_link_3: mass 0.006444241316270568 -> 0.010740402193784278; geometry collision box size=0.03916666666666666 0.028 0.0009; visual box size=0.03916666666666666 0.028 0.0009
- link finger_1_segment_link_4: mass 0.006444241316270568 -> 0.010740402193784278; geometry collision box size=0.03916666666666666 0.028 0.0009; visual box size=0.03916666666666666 0.028 0.0009
- link finger_1_segment_link_5: mass 0.006444241316270568 -> 0.010740402193784278; geometry collision box size=0.03916666666666666 0.028 0.0009; visual box size=0.03916666666666666 0.028 0.0009
- link finger_1_segment_link_6: mass 0.006444241316270568 -> 0.010740402193784278; geometry collision box size=0.03916666666666666 0.028 0.0009; visual box size=0.03916666666666666 0.028 0.0009
- link finger_2_finger_hook_link: mass 0.006444241316270568 -> 0.010740402193784278
- link finger_2_segment_link_1: mass 0.006444241316270568 -> 0.010740402193784278; geometry collision box size=0.03916666666666666 0.028 0.0009; visual box size=0.03916666666666666 0.028 0.0009
- link finger_2_segment_link_2: mass 0.006444241316270568 -> 0.010740402193784278; geometry collision box size=0.03916666666666666 0.028 0.0009; visual box size=0.03916666666666666 0.028 0.0009
- link finger_2_segment_link_3: mass 0.006444241316270568 -> 0.010740402193784278; geometry collision box size=0.03916666666666666 0.028 0.0009; visual box size=0.03916666666666666 0.028 0.0009
- link finger_2_segment_link_4: mass 0.006444241316270568 -> 0.010740402193784278; geometry collision box size=0.03916666666666666 0.028 0.0009; visual box size=0.03916666666666666 0.028 0.0009
- link finger_2_segment_link_5: mass 0.006444241316270568 -> 0.010740402193784278; geometry collision box size=0.03916666666666666 0.028 0.0009; visual box size=0.03916666666666666 0.028 0.0009
- link finger_2_segment_link_6: mass 0.006444241316270568 -> 0.010740402193784278; geometry collision box size=0.03916666666666666 0.028 0.0009; visual box size=0.03916666666666666 0.028 0.0009
- link finger_3_finger_hook_link: mass 0.006444241316270568 -> 0.010740402193784278
- link finger_3_segment_link_1: mass 0.006444241316270568 -> 0.010740402193784278; geometry collision box size=0.03916666666666666 0.028 0.0009; visual box size=0.03916666666666666 0.028 0.0009
- link finger_3_segment_link_2: mass 0.006444241316270568 -> 0.010740402193784278; geometry collision box size=0.03916666666666666 0.028 0.0009; visual box size=0.03916666666666666 0.028 0.0009
- link finger_3_segment_link_3: mass 0.006444241316270568 -> 0.010740402193784278; geometry collision box size=0.03916666666666666 0.028 0.0009; visual box size=0.03916666666666666 0.028 0.0009
- link finger_3_segment_link_4: mass 0.006444241316270568 -> 0.010740402193784278; geometry collision box size=0.03916666666666666 0.028 0.0009; visual box size=0.03916666666666666 0.028 0.0009
- link finger_3_segment_link_5: mass 0.006444241316270568 -> 0.010740402193784278; geometry collision box size=0.03916666666666666 0.028 0.0009; visual box size=0.03916666666666666 0.028 0.0009
- link finger_3_segment_link_6: mass 0.006444241316270568 -> 0.010740402193784278; geometry collision box size=0.03916666666666666 0.028 0.0009; visual box size=0.03916666666666666 0.028 0.0009
Joints:
- removed joint finger_1_segment_joint_6
- removed joint finger_1_segment_joint_7
- removed joint finger_1_segment_joint_8
- removed joint finger_1_segment_joint_9
- removed joint finger_2_segment_joint_6
- removed joint finger_2_segment_joint_7
- removed joint finger_2_segment_joint_8
- removed joint finger_2_segment_joint_9
- removed joint finger_3_segment_joint_6
- removed joint finger_3_segment_joint_7
- removed joint finger_3_segment_joint_8
- removed joint finger_3_segment_joint_9
- joint finger_1_finger_hook_joint: origin xyz=0.0235 0 0 rpy=0 -1.5707963267948502 0 -> xyz=0.03916666666666666 0 0 rpy=0 -1.5707963267948502 0; parent finger_1_segment_link_10 -> finger_1_segment_link_6
- joint finger_1_segment_joint_1: origin xyz=0.0235 0 0 rpy=0 0 0 -> xyz=0.03916666666666666 0 0 rpy=0 0 0
- joint finger_1_segment_joint_2: origin xyz=0.0235 0 0 rpy=0 0 0 -> xyz=0.03916666666666666 0 0 rpy=0 0 0
- joint finger_1_segment_joint_3: origin xyz=0.0235 0 0 rpy=0 0 0 -> xyz=0.03916666666666666 0 0 rpy=0 0 0
- joint finger_1_segment_joint_4: origin xyz=0.0235 0 0 rpy=0 0 0 -> xyz=0.03916666666666666 0 0 rpy=0 0 0
- joint finger_1_segment_joint_5: origin xyz=0.0235 0 0 rpy=0 0 0 -> xyz=0.03916666666666666 0 0 rpy=0 0 0
- joint finger_2_finger_hook_joint: origin xyz=0.0235 0 0 rpy=0 -1.5707963267948502 0 -> xyz=0.03916666666666666 0 0 rpy=0 -1.5707963267948502 0; parent finger_2_segment_link_10 -> finger_2_segment_link_6
- joint finger_2_segment_joint_1: origin xyz=0.0235 0 0 rpy=0 0 0 -> xyz=0.03916666666666666 0 0 rpy=0 0 0
- joint finger_2_segment_joint_2: origin xyz=0.0235 0 0 rpy=0 0 0 -> xyz=0.03916666666666666 0 0 rpy=0 0 0
- joint finger_2_segment_joint_3: origin xyz=0.0235 0 0 rpy=0 0 0 -> xyz=0.03916666666666666 0 0 rpy=0 0 0
- joint finger_2_segment_joint_4: origin xyz=0.0235 0 0 rpy=0 0 0 -> xyz=0.03916666666666666 0 0 rpy=0 0 0
- joint finger_2_segment_joint_5: origin xyz=0.0235 0 0 rpy=0 0 0 -> xyz=0.03916666666666666 0 0 rpy=0 0 0
- joint finger_3_finger_hook_joint: origin xyz=0.0235 0 0 rpy=0 -1.5707963267948502 0 -> xyz=0.03916666666666666 0 0 rpy=0 -1.5707963267948502 0; parent finger_3_segment_link_10 -> finger_3_segment_link_6
- joint finger_3_segment_joint_1: origin xyz=0.0235 0 0 rpy=0 0 0 -> xyz=0.03916666666666666 0 0 rpy=0 0 0
- joint finger_3_segment_joint_2: origin xyz=0.0235 0 0 rpy=0 0 0 -> xyz=0.03916666666666666 0 0 rpy=0 0 0
- joint finger_3_segment_joint_3: origin xyz=0.0235 0 0 rpy=0 0 0 -> xyz=0.03916666666666666 0 0 rpy=0 0 0
- joint finger_3_segment_joint_4: origin xyz=0.0235 0 0 rpy=0 0 0 -> xyz=0.03916666666666666 0 0 rpy=0 0 0
- joint finger_3_segment_joint_5: origin xyz=0.0235 0 0 rpy=0 0 0 -> xyz=0.03916666666666666 0 0 rpy=0 0 0

File: mujoco/urdf/gripper_task.urdf (robot description, URDF)
Before this commit: robot gripper_task, 42 links, 41 joints
Links:
- removed link finger_1_segment_link_10
- removed link finger_1_segment_link_7
- removed link finger_1_segment_link_8
- removed link finger_1_segment_link_9
- removed link finger_2_segment_link_10
- removed link finger_2_segment_link_7
- removed link finger_2_segment_link_8
- removed link finger_2_segment_link_9
- removed link finger_3_segment_link_10
- removed link finger_3_segment_link_7
- removed link finger_3_segment_link_8
- removed link finger_3_segment_link_9
- link finger_1_finger_hook_link: mass 0.006444241316270568 -> 0.010740402193784278
- link finger_1_segment_link_1: mass 0.006444241316270568 -> 0.010740402193784278; geometry collision box size=0.03916666666666666 0.028 0.0009; visual box size=0.03916666666666666 0.028 0.0009
- link finger_1_segment_link_2: mass 0.006444241316270568 -> 0.010740402193784278; geometry collision box size=0.03916666666666666 0.028 0.0009; visual box size=0.03916666666666666 0.028 0.0009
- link finger_1_segment_link_3: mass 0.006444241316270568 -> 0.010740402193784278; geometry collision box size=0.03916666666666666 0.028 0.0009; visual box size=0.03916666666666666 0.028 0.0009
- link finger_1_segment_link_4: mass 0.006444241316270568 -> 0.010740402193784278; geometry collision box size=0.03916666666666666 0.028 0.0009; visual box size=0.03916666666666666 0.028 0.0009
- link finger_1_segment_link_5: mass 0.006444241316270568 -> 0.010740402193784278; geometry collision box size=0.03916666666666666 0.028 0.0009; visual box size=0.03916666666666666 0.028 0.0009
- link finger_1_segment_link_6: mass 0.006444241316270568 -> 0.010740402193784278; geometry collision box size=0.03916666666666666 0.028 0.0009; visual box size=0.03916666666666666 0.028 0.0009
- link finger_2_finger_hook_link: mass 0.006444241316270568 -> 0.010740402193784278
- link finger_2_segment_link_1: mass 0.006444241316270568 -> 0.010740402193784278; geometry collision box size=0.03916666666666666 0.028 0.0009; visual box size=0.03916666666666666 0.028 0.0009
- link finger_2_segment_link_2: mass 0.006444241316270568 -> 0.010740402193784278; geometry collision box size=0.03916666666666666 0.028 0.0009; visual box size=0.03916666666666666 0.028 0.0009
- link finger_2_segment_link_3: mass 0.006444241316270568 -> 0.010740402193784278; geometry collision box size=0.03916666666666666 0.028 0.0009; visual box size=0.03916666666666666 0.028 0.0009
- link finger_2_segment_link_4: mass 0.006444241316270568 -> 0.010740402193784278; geometry collision box size=0.03916666666666666 0.028 0.0009; visual box size=0.03916666666666666 0.028 0.0009
- link finger_2_segment_link_5: mass 0.006444241316270568 -> 0.010740402193784278; geometry collision box size=0.03916666666666666 0.028 0.0009; visual box size=0.03916666666666666 0.028 0.0009
- link finger_2_segment_link_6: mass 0.006444241316270568 -> 0.010740402193784278; geometry collision box size=0.03916666666666666 0.028 0.0009; visual box size=0.03916666666666666 0.028 0.0009
- link finger_3_finger_hook_link: mass 0.006444241316270568 -> 0.010740402193784278
- link finger_3_segment_link_1: mass 0.006444241316270568 -> 0.010740402193784278; geometry collision box size=0.03916666666666666 0.028 0.0009; visual box size=0.03916666666666666 0.028 0.0009
- link finger_3_segment_link_2: mass 0.006444241316270568 -> 0.010740402193784278; geometry collision box size=0.03916666666666666 0.028 0.0009; visual box size=0.03916666666666666 0.028 0.0009
- link finger_3_segment_link_3: mass 0.006444241316270568 -> 0.010740402193784278; geometry collision box size=0.03916666666666666 0.028 0.0009; visual box size=0.03916666666666666 0.028 0.0009
- link finger_3_segment_link_4: mass 0.006444241316270568 -> 0.010740402193784278; geometry collision box size=0.03916666666666666 0.028 0.0009; visual box size=0.03916666666666666 0.028 0.0009
- link finger_3_segment_link_5: mass 0.006444241316270568 -> 0.010740402193784278; geometry collision box size=0.03916666666666666 0.028 0.0009; visual box size=0.03916666666666666 0.028 0.0009
- link finger_3_segment_link_6: mass 0.006444241316270568 -> 0.010740402193784278; geometry collision box size=0.03916666666666666 0.028 0.0009; visual box size=0.03916666666666666 0.028 0.0009
Joints:
- removed joint finger_1_segment_joint_6
- removed joint finger_1_segment_joint_7
- removed joint finger_1_segment_joint_8
- removed joint finger_1_segment_joint_9
- removed joint finger_2_segment_joint_6
- removed joint finger_2_segment_joint_7
- removed joint finger_2_segment_joint_8
- removed joint finger_2_segment_joint_9
- removed joint finger_3_segment_joint_6
- removed joint finger_3_segment_joint_7
- removed joint finger_3_segment_joint_8
- removed joint finger_3_segment_joint_9
- joint finger_1_finger_hook_joint: origin xyz=0.0235 0 0 rpy=0 -1.5707963267948502 0 -> xyz=0.03916666666666666 0 0 rpy=0 -1.5707963267948502 0; parent finger_1_segment_link_10 -> finger_1_segment_link_6
- joint finger_1_segment_joint_1: origin xyz=0.0235 0 0 rpy=0 0 0 -> xyz=0.03916666666666666 0 0 rpy=0 0 0
- joint finger_1_segment_joint_2: origin xyz=0.0235 0 0 rpy=0 0 0 -> xyz=0.03916666666666666 0 0 rpy=0 0 0
- joint finger_1_segment_joint_3: origin xyz=0.0235 0 0 rpy=0 0 0 -> xyz=0.03916666666666666 0 0 rpy=0 0 0
- joint finger_1_segment_joint_4: origin xyz=0.0235 0 0 rpy=0 0 0 -> xyz=0.03916666666666666 0 0 rpy=0 0 0
- joint finger_1_segment_joint_5: origin xyz=0.0235 0 0 rpy=0 0 0 -> xyz=0.03916666666666666 0 0 rpy=0 0 0
- joint finger_2_finger_hook_joint: origin xyz=0.0235 0 0 rpy=0 -1.5707963267948502 0 -> xyz=0.03916666666666666 0 0 rpy=0 -1.5707963267948502 0; parent finger_2_segment_link_10 -> finger_2_segment_link_6
- joint finger_2_segment_joint_1: origin xyz=0.0235 0 0 rpy=0 0 0 -> xyz=0.03916666666666666 0 0 rpy=0 0 0
- joint finger_2_segment_joint_2: origin xyz=0.0235 0 0 rpy=0 0 0 -> xyz=0.03916666666666666 0 0 rpy=0 0 0
- joint finger_2_segment_joint_3: origin xyz=0.0235 0 0 rpy=0 0 0 -> xyz=0.03916666666666666 0 0 rpy=0 0 0
- joint finger_2_segment_joint_4: origin xyz=0.0235 0 0 rpy=0 0 0 -> xyz=0.03916666666666666 0 0 rpy=0 0 0
- joint finger_2_segment_joint_5: origin xyz=0.0235 0 0 rpy=0 0 0 -> xyz=0.03916666666666666 0 0 rpy=0 0 0
- joint finger_3_finger_hook_joint: origin xyz=0.0235 0 0 rpy=0 -1.5707963267948502 0 -> xyz=0.03916666666666666 0 0 rpy=0 -1.5707963267948502 0; parent finger_3_segment_link_10 -> finger_3_segment_link_6
- joint finger_3_segment_joint_1: origin xyz=0.0235 0 0 rpy=0 0 0 -> xyz=0.03916666666666666 0 0 rpy=0 0 0
- joint finger_3_segment_joint_2: origin xyz=0.0235 0 0 rpy=0 0 0 -> xyz=0.03916666666666666 0 0 rpy=0 0 0
- joint finger_3_segment_joint_3: origin xyz=0.0235 0 0 rpy=0 0 0 -> xyz=0.03916666666666666 0 0 rpy=0 0 0
- joint finger_3_segment_joint_4: origin xyz=0.0235 0 0 rpy=0 0 0 -> xyz=0.03916666666666666 0 0 rpy=0 0 0
- joint finger_3_segment_joint_5: origin xyz=0.0235 0 0 rpy=0 0 0 -> xyz=0.03916666666666666 0 0 rpy=0 0 0

File: mujoco/urdf/panda_and_gripper_mujoco.urdf (robot description, URDF)
Before this commit: robot panda_and_gripper, 51 links, 50 joints
Links:
- removed link finger_1_segment_link_10
- removed link finger_1_segment_link_7
- removed link finger_1_segment_link_8
- removed link finger_1_segment_link_9
- removed link finger_2_segment_link_10
- removed link finger_2_segment_link_7
- removed link finger_2_segment_link_8
- removed link finger_2_segment_link_9
- removed link finger_3_segment_link_10
- removed link finger_3_segment_link_7
- removed link finger_3_segment_link_8
- removed link finger_3_segment_link_9
- link finger_1_finger_hook_link: mass 0.006444241316270568 -> 0.010740402193784278
- link finger_1_segment_link_1: mass 0.006444241316270568 -> 0.010740402193784278; geometry collision box size=0.03916666666666666 0.028 0.0009; visual box size=0.03916666666666666 0.028 0.0009
- link finger_1_segment_link_2: mass 0.006444241316270568 -> 0.010740402193784278; geometry collision box size=0.03916666666666666 0.028 0.0009; visual box size=0.03916666666666666 0.028 0.0009
- link finger_1_segment_link_3: mass 0.006444241316270568 -> 0.010740402193784278; geometry collision box size=0.03916666666666666 0.028 0.0009; visual box size=0.03916666666666666 0.028 0.0009
- link finger_1_segment_link_4: mass 0.006444241316270568 -> 0.010740402193784278; geometry collision box size=0.03916666666666666 0.028 0.0009; visual box size=0.03916666666666666 0.028 0.0009
- link finger_1_segment_link_5: mass 0.006444241316270568 -> 0.010740402193784278; geometry collision box size=0.03916666666666666 0.028 0.0009; visual box size=0.03916666666666666 0.028 0.0009
- link finger_1_segment_link_6: mass 0.006444241316270568 -> 0.010740402193784278; geometry collision box size=0.03916666666666666 0.028 0.0009; visual box size=0.03916666666666666 0.028 0.0009
- link finger_2_finger_hook_link: mass 0.006444241316270568 -> 0.010740402193784278
- link finger_2_segment_link_1: mass 0.006444241316270568 -> 0.010740402193784278; geometry collision box size=0.03916666666666666 0.028 0.0009; visual box size=0.03916666666666666 0.028 0.0009
- link finger_2_segment_link_2: mass 0.006444241316270568 -> 0.010740402193784278; geometry collision box size=0.03916666666666666 0.028 0.0009; visual box size=0.03916666666666666 0.028 0.0009
- link finger_2_segment_link_3: mass 0.006444241316270568 -> 0.010740402193784278; geometry collision box size=0.03916666666666666 0.028 0.0009; visual box size=0.03916666666666666 0.028 0.0009
- link finger_2_segment_link_4: mass 0.006444241316270568 -> 0.010740402193784278; geometry collision box size=0.03916666666666666 0.028 0.0009; visual box size=0.03916666666666666 0.028 0.0009
- link finger_2_segment_link_5: mass 0.006444241316270568 -> 0.010740402193784278; geometry collision box size=0.03916666666666666 0.028 0.0009; visual box size=0.03916666666666666 0.028 0.0009
- link finger_2_segment_link_6: mass 0.006444241316270568 -> 0.010740402193784278; geometry collision box size=0.03916666666666666 0.028 0.0009; visual box size=0.03916666666666666 0.028 0.0009
- link finger_3_finger_hook_link: mass 0.006444241316270568 -> 0.010740402193784278
- link finger_3_segment_link_1: mass 0.006444241316270568 -> 0.010740402193784278; geometry collision box size=0.03916666666666666 0.028 0.0009; visual box size=0.03916666666666666 0.028 0.0009
- link finger_3_segment_link_2: mass 0.006444241316270568 -> 0.010740402193784278; geometry collision box size=0.03916666666666666 0.028 0.0009; visual box size=0.03916666666666666 0.028 0.0009
- link finger_3_segment_link_3: mass 0.006444241316270568 -> 0.010740402193784278; geometry collision box size=0.03916666666666666 0.028 0.0009; visual box size=0.03916666666666666 0.028 0.0009
- link finger_3_segment_link_4: mass 0.006444241316270568 -> 0.010740402193784278; geometry collision box size=0.03916666666666666 0.028 0.0009; visual box size=0.03916666666666666 0.028 0.0009
- link finger_3_segment_link_5: mass 0.006444241316270568 -> 0.010740402193784278; geometry collision box size=0.03916666666666666 0.028 0.0009; visual box size=0.03916666666666666 0.028 0.0009
- link finger_3_segment_link_6: mass 0.006444241316270568 -> 0.010740402193784278; geometry collision box size=0.03916666666666666 0.028 0.0009; visual box size=0.03916666666666666 0.028 0.0009
Joints:
- removed joint finger_1_segment_joint_6
- removed joint finger_1_segment_joint_7
- removed joint finger_1_segment_joint_8
- removed joint finger_1_segment_joint_9
- removed joint finger_2_segment_joint_6
- removed joint finger_2_segment_joint_7
- removed joint finger_2_segment_joint_8
- removed joint finger_2_segment_joint_9
- removed joint finger_3_segment_joint_6
- removed joint finger_3_segment_joint_7
- removed joint finger_3_segment_joint_8
- removed joint finger_3_segment_joint_9
- joint finger_1_finger_hook_joint: origin xyz=0.0235 0 0 rpy=0 -1.5707963267948502 0 -> xyz=0.03916666666666666 0 0 rpy=0 -1.5707963267948502 0; parent finger_1_segment_link_10 -> finger_1_segment_link_6
- joint finger_1_segment_joint_1: origin xyz=0.0235 0 0 rpy=0 0 0 -> xyz=0.03916666666666666 0 0 rpy=0 0 0
- joint finger_1_segment_joint_2: origin xyz=0.0235 0 0 rpy=0 0 0 -> xyz=0.03916666666666666 0 0 rpy=0 0 0
- joint finger_1_segment_joint_3: origin xyz=0.0235 0 0 rpy=0 0 0 -> xyz=0.03916666666666666 0 0 rpy=0 0 0
- joint finger_1_segment_joint_4: origin xyz=0.0235 0 0 rpy=0 0 0 -> xyz=0.03916666666666666 0 0 rpy=0 0 0
- joint finger_1_segment_joint_5: origin xyz=0.0235 0 0 rpy=0 0 0 -> xyz=0.03916666666666666 0 0 rpy=0 0 0
- joint finger_2_finger_hook_joint: origin xyz=0.0235 0 0 rpy=0 -1.5707963267948502 0 -> xyz=0.03916666666666666 0 0 rpy=0 -1.5707963267948502 0; parent finger_2_segment_link_10 -> finger_2_segment_link_6
- joint finger_2_segment_joint_1: origin xyz=0.0235 0 0 rpy=0 0 0 -> xyz=0.03916666666666666 0 0 rpy=0 0 0
- joint finger_2_segment_joint_2: origin xyz=0.0235 0 0 rpy=0 0 0 -> xyz=0.03916666666666666 0 0 rpy=0 0 0
- joint finger_2_segment_joint_3: origin xyz=0.0235 0 0 rpy=0 0 0 -> xyz=0.03916666666666666 0 0 rpy=0 0 0
- joint finger_2_segment_joint_4: origin xyz=0.0235 0 0 rpy=0 0 0 -> xyz=0.03916666666666666 0 0 rpy=0 0 0
- joint finger_2_segment_joint_5: origin xyz=0.0235 0 0 rpy=0 0 0 -> xyz=0.03916666666666666 0 0 rpy=0 0 0
- joint finger_3_finger_hook_joint: origin xyz=0.0235 0 0 rpy=0 -1.5707963267948502 0 -> xyz=0.03916666666666666 0 0 rpy=0 -1.5707963267948502 0; parent finger_3_segment_link_10 -> finger_3_segment_link_6
- joint finger_3_segment_joint_1: origin xyz=0.0235 0 0 rpy=0 0 0 -> xyz=0.03916666666666666 0 0 rpy=0 0 0
- joint finger_3_segment_joint_2: origin xyz=0.0235 0 0 rpy=0 0 0 -> xyz=0.03916666666666666 0 0 rpy=0 0 0
- joint finger_3_segment_joint_3: origin xyz=0.0235 0 0 rpy=0 0 0 -> xyz=0.03916666666666666 0 0 rpy=0 0 0
- joint finger_3_segment_joint_4: origin xyz=0.0235 0 0 rpy=0 0 0 -> xyz=0.03916666666666666 0 0 rpy=0 0 0
- joint finger_3_segment_joint_5: origin xyz=0.0235 0 0 rpy=0 0 0 -> xyz=0.03916666666666666 0 0 rpy=0 0 0
