Commit message: add UDL and fixed rev joint

File: xacro/gripper.main.xacro (robot description, xacro)
@@ -13,4 +13,6 @@
     <xacro:property name="finger_angle_min" value="${-1 * yaml_dict['gripper_params']['angle_max_abs']}"/>
     <xacro:property name="finger_angle_max" value="${yaml_dict['gripper_params']['angle_max_abs']}"/>
+    <!-- testing -->
+    <xacro:property name="fixed_rev_joint" value="${yaml_dict['gripper_config']['fixed_rev_joint']}"/>
   	<!-- PARAMETERS TO BE SET BY HAND -->
     <!-- Define limits of each joint, these all in SI units -->
@@ -170,15 +172,24 @@
       </joint>
       <!-- Revolute joint -->
-      <joint name="finger_${number}_revolute_joint" type="revolute">
-        <axis xyz="0 0 1" rpy="0 0 0"/>
-        <parent link="finger_${number}_intermediate"/>
-        <child link="finger_${number}"/>
-        <xacro:finger_origin number="${number}"/>
-        <limit effort="${limit_effort_revolute}"
-        			 lower="${finger_angle_min}"
-        			 upper="${finger_angle_max}"
-        			 velocity="${finger_angle_velocity}"/>
-        <dynamics damping="${joint_damping}"/>
-      </joint>
+      <xacro:if value="${fixed_rev_joint}">
+        <joint name="finger_${number}_revolute_joint" type="fixed">
+          <parent link="finger_${number}_intermediate"/>
+          <child link="finger_${number}"/>
+          <xacro:finger_origin number="${number}"/>
+        </joint>
+      </xacro:if>
+      <xacro:if value="${not fixed_rev_joint}">
+        <joint name="finger_${number}_revolute_joint" type="revolute">
+          <axis xyz="0 0 1" rpy="0 0 0"/>
+          <parent link="finger_${number}_intermediate"/>
+          <child link="finger_${number}"/>
+          <xacro:finger_origin number="${number}"/>
+          <limit effort="${limit_effort_revolute}"
+                lower="${finger_angle_min}"
+                upper="${finger_angle_max}"
+                velocity="${finger_angle_velocity}"/>
+          <dynamics damping="${joint_damping}"/>
+        </joint>
+      </xacro:if>
     </xacro:macro>
     <!-- FINGERS -->

Commit message: test adjustments for testing set

File: xacro/gripper.main.xacro (robot description, xacro)
@@ -160,15 +160,30 @@
       </link>
       <!-- Prismatic joint -->
-      <joint name="finger_${number}_prismatic_joint" type="prismatic">
-        <axis xyz="0 1 0" rpy="0 0 0"/>
-        <parent link="gripper_base_link"/>
-        <child link="finger_${number}_intermediate"/>
-        <xacro:finger_intermediate_origin number="${number}"/>
-        <limit effort="${limit_effort_prismatic}"
-        			 lower="${finger_displacement_min}"
-        			 upper="${finger_displacement_max}"
-        			 velocity="${finger_displacement_velocity}"/>
-        <dynamics damping="${joint_damping}"/>
-      </joint>
+      <xacro:if value="${fixed_rev_joint}">
+        <joint name="finger_${number}_prismatic_joint" type="fixed">
+          <parent link="gripper_base_link"/>
+          <child link="finger_${number}_intermediate"/>
+          <!-- <xacro:finger_intermediate_origin number="${number}"/> -->
+          <origin xyz="${100e-3 * sin((number-1)*((2*pi)/3))}
+                       ${100e-3 * cos((number-1)*((2*pi)/3))}
+                       0"
+                  rpy="${3*pi/2}
+                       ${3*pi/2}
+                       ${(pi/2) - (number-1)*(2*pi/3)}" />
+        </joint>
+      </xacro:if>
+      <xacro:if value="${not fixed_rev_joint}">
+        <joint name="finger_${number}_prismatic_joint" type="prismatic">
+          <axis xyz="0 1 0" rpy="0 0 0"/>
+          <parent link="gripper_base_link"/>
+          <child link="finger_${number}_intermediate"/>
+          <xacro:finger_intermediate_origin number="${number}"/>
+          <limit effort="${limit_effort_prismatic}"
+                lower="${finger_displacement_min}"
+                upper="${finger_displacement_max}"
+                velocity="${finger_displacement_velocity}"/>
+          <dynamics damping="${joint_damping}"/>
+        </joint>
+      </xacro:if>
       <!-- Revolute joint -->
       <xacro:if value="${fixed_rev_joint}">

File: xacro/gripper.segmented_fingers.xacro (robot description, xacro)
@@ -247,5 +247,6 @@
 		          upper="1.0"
 		          velocity="1.0"/>
-		    <dynamics damping="${joint_damping}" friction="${joint_friction}"/>
+        <!-- give extra damping/friction to stop unwanted movement -->
+		    <dynamics damping="100" friction="100"/>
       </joint>
     </xacro:if>

Commit message: minor streamlines, fixes

File: xacro/gripper.main.xacro (robot description, xacro)
@@ -13,6 +13,5 @@
     <xacro:property name="finger_angle_min" value="${-1 * yaml_dict['gripper_params']['angle_max_abs']}"/>
     <xacro:property name="finger_angle_max" value="${yaml_dict['gripper_params']['angle_max_abs']}"/>
-    <!-- testing -->
-    <xacro:property name="fixed_rev_joint" value="${yaml_dict['gripper_config']['fixed_rev_joint']}"/>
+    <xacro:property name="fixed_motor_joints" value="${yaml_dict['gripper_config']['fixed_motor_joints']}"/>
   	<!-- PARAMETERS TO BE SET BY HAND -->
     <!-- Define limits of each joint, these all in SI units -->
@@ -160,5 +159,5 @@
       </link>
       <!-- Prismatic joint -->
-      <xacro:if value="${fixed_rev_joint}">
+      <xacro:if value="${fixed_motor_joints}">
         <joint name="finger_${number}_prismatic_joint" type="fixed">
           <parent link="gripper_base_link"/>
@@ -173,5 +172,5 @@
         </joint>
       </xacro:if>
-      <xacro:if value="${not fixed_rev_joint}">
+      <xacro:if value="${not fixed_motor_joints}">
         <joint name="finger_${number}_prismatic_joint" type="prismatic">
           <axis xyz="0 1 0" rpy="0 0 0"/>
@@ -187,5 +186,5 @@
       </xacro:if>
       <!-- Revolute joint -->
-      <xacro:if value="${fixed_rev_joint}">
+      <xacro:if value="${fixed_motor_joints}">
         <joint name="finger_${number}_revolute_joint" type="fixed">
           <parent link="finger_${number}_intermediate"/>
@@ -194,5 +193,5 @@
         </joint>
       </xacro:if>
-      <xacro:if value="${not fixed_rev_joint}">
+      <xacro:if value="${not fixed_motor_joints}">
         <joint name="finger_${number}_revolute_joint" type="revolute">
           <axis xyz="0 0 1" rpy="0 0 0"/>
