Commit message: fix 7mm offset and new gear ratio

File: xacro/gripper.xacro (robot description, xacro)
@@ -4,7 +4,6 @@
 		<!-- PARAMETERS TO BE SET BY HAND -->
 		<!-- xyz values to connect the segmented finger to the finger platform -->
-		<!-- TODO verfiy these values -->
 		<xacro:property name="x_fix" value="0.129"/>
-		<xacro:property name="y_fix" value="-0.007"/>
+		<xacro:property name="y_fix" value="0"/>
 		<xacro:property name="z_fix" value="0"/>
 		<!-- END OF PARAMETERS TO BE SET BY HAND -->
