Commit message: finish adding auto generation

File: mujoco/xacro/gripper_task.urdf.xacro (robot description, xacro)
@@ -8,4 +8,7 @@
 	<!-- extract the gripper config information -->
 	<xacro:property name="xy_base_joint" value="${yaml_dict['gripper_config']['xy_base_joint']}"/>
+	<xacro:property name="fingertip_clearance" value="${yaml_dict['gripper_params']['fingertip_clearance']}"/>
+	<xacro:property name="hook_length" value="${yaml_dict['gripper_params']['hook_length']}"/>
+	<xacro:property name="hook_angle_rad" value="${yaml_dict['gripper_params']['hook_angle_degrees'] * (3.141592 / 180.0)}"/>
   <!-- include the mujoco settings xacro -->
 	<xacro:include filename="${path_to_top}/mujoco/xacro/mujoco.xacro"/>
@@ -17,8 +20,17 @@
 	past that. Note that this height is calibrated manually using mujoco and with
   checking the wrist z sensor for contact. This is calibrated AFTER the gripper
-	has settled (ie joint controller stiffness accounted for)-->
-	<xacro:property name="fingertip_touches_ground" value="0.376"/>
-	<xacro:property name="fingertip_clearance" value="0.01"/>
-	<xacro:property name="h" value="${fingertip_touches_ground + fingertip_clearance}"/>
+	has settled (ie joint controller stiffness accounted for). See the function
+	'calibrate_reset()' in myfunctions.cpp and turn on debug mode to see the final
+	settled finger end height above the ground, you can use this to adjust the value
+	of 'fingerend_touches_ground' so that a 'fingertip_clearance' of 0.0 gives a
+	finger end height of 0.0 -->
+	<xacro:property name="fingerend_touches_ground" value="${0.1407 + yaml_dict['gripper_params']['finger_length']}"/>
+	<xacro:if value="${yaml_dict['gripper_params']['hook_angle_degrees'] > 90}">
+		<xacro:property name="hook_extra" value="0.0"/>
+	</xacro:if>
+	<xacro:if value="${not (yaml_dict['gripper_params']['hook_angle_degrees'] > 90)}">
+		<xacro:property name="hook_extra" value="${hook_length * cos(hook_angle_rad)}"/>
+	</xacro:if>
+	<xacro:property name="h" value="${fingerend_touches_ground + fingertip_clearance + hook_extra}"/>
   <!-- create gripper base joints in mujoco -->
 	<xacro:if value="${xy_base_joint}">

Commit message: fix for ubuntu 20 - rm xacro.load_yaml

File: mujoco/xacro/gripper_task.urdf.xacro (robot description, xacro)
@@ -5,5 +5,5 @@
 	<!-- load the gripper config information -->
 	<xacro:property name="filename" value="${path_to_top}/config/gripper.yaml"/>
-	<xacro:property name="yaml_dict" value="${xacro.load_yaml(filename)}"/>
+	<xacro:property name="yaml_dict" value="${load_yaml(filename)}"/>
 	<!-- extract the gripper config information -->
 	<xacro:property name="xy_base_joint" value="${yaml_dict['gripper_config']['xy_base_joint']}"/>

File: xacro/gripper.main.xacro (robot description, xacro)
@@ -4,5 +4,5 @@
 		<!-- load the gripper config information -->
     <xacro:property name="filename" value="${path_to_top}/config/gripper.yaml"/>
-    <xacro:property name="yaml_dict" value="${xacro.load_yaml(filename)}"/>
+    <xacro:property name="yaml_dict" value="${load_yaml(filename)}"/>
     <!-- extract the gripper config information -->
     <xacro:property name="is_segmented" value="${yaml_dict['gripper_config']['is_segmented']}"/>

File: xacro/gripper.xacro (robot description, xacro)
@@ -14,5 +14,5 @@
 		<xacro:include filename="${path_to_top}/xacro/gripper.segmented_fingers.xacro"/>
 		<!-- load information from the gripper yaml file -->
-		<xacro:property name="yaml_dict" value="${xacro.load_yaml(filename)}"/>
+		<xacro:property name="yaml_dict" value="${load_yaml(filename)}"/>
 		<xacro:property name="is_segmented" value="${yaml_dict['gripper_config']['is_segmented']}"/>
 		<!-- create instance of gripper -->

Commit message: align xml base Y motion with mujoco Y axis

File: mujoco/xacro/gripper_task.urdf.xacro (robot description, xacro)
@@ -62,5 +62,5 @@
 		<joint name="base_Y_joint" type="prismatic">
 			<origin xyz="0 0 0" rpy="0 0 0"/>
-			<axis xyz="0 1 0" rpy="0 0 0"/>
+			<axis xyz="0 -1 0" rpy="$0 0 0"/>
 			<parent link="base_XY"/>
 			<child link="base_YZ"/>

Commit message: add gripper yaw action

File: mujoco/xacro/gripper_task.urdf.xacro (robot description, xacro)
@@ -8,4 +8,5 @@
 	<!-- extract the gripper config information -->
 	<xacro:property name="xy_base_joint" value="${yaml_dict['gripper_config']['xy_base_joint']}"/>
+	<xacro:property name="z_base_rotation" value="${yaml_dict['gripper_config']['z_base_rotation']}"/>
 	<xacro:property name="fingertip_clearance" value="${yaml_dict['gripper_params']['fingertip_clearance']}"/>
 	<xacro:property name="hook_length" value="${yaml_dict['gripper_params']['hook_length']}"/>
@@ -71,15 +72,47 @@
 			<dynamics damping="1"/>
 		</joint>
-		<joint name="base_Z_joint" type="prismatic">
-			<origin xyz="0 0 0" rpy="0 0 0"/>
-			<axis xyz="0 0 1" rpy="0 0 0"/>
-			<parent link="base_YZ"/>
-			<child link="gripper_base_link"/>
-			<limit effort="1e3"
-						lower="-1"
-						upper="1"
-						velocity="1"/>
-			<dynamics damping="1"/>
-		</joint>
+		<xacro:if value="${z_base_rotation}">
+			<link name="base_ZrotZ">
+				<inertial>
+					<mass value="1.0"/>
+					<inertia ixx="1e-3" ixy="0" ixz="0" iyy="1e-3" iyz="0" izz="1e-3"/>
+				</inertial>
+			</link>
+			<joint name="base_Z_joint" type="prismatic">
+				<origin xyz="0 0 0" rpy="0 0 0"/>
+				<axis xyz="0 0 1" rpy="0 0 0"/>
+				<parent link="base_YZ"/>
+				<child link="base_ZrotZ"/>
+				<limit effort="1e3"
+							lower="-1"
+							upper="1"
+							velocity="1"/>
+				<dynamics damping="1"/>
+			</joint>
+			<joint name="base_Z_rotation_joint" type="revolute">
+				<origin xyz="0 0 0" rpy="0 0 0"/>
+				<axis xyz="0 0 1" rpy="0 0 0"/>
+				<parent link="base_ZrotZ"/>
+				<child link="gripper_base_link"/>
+				<limit effort="1e3"
+							lower="-1000"
+							upper="1000"
+							velocity="1"/>
+				<dynamics damping="1"/>
+			</joint>
+		</xacro:if>
+		<xacro:if value="${not z_base_rotation}">
+			<joint name="base_Z_joint" type="prismatic">
+				<origin xyz="0 0 0" rpy="0 0 0"/>
+				<axis xyz="0 0 1" rpy="0 0 0"/>
+				<parent link="base_YZ"/>
+				<child link="gripper_base_link"/>
+				<limit effort="1e3"
+							lower="-1"
+							upper="1"
+							velocity="1"/>
+				<dynamics damping="1"/>
+			</joint>
+		</xacro:if>
 	</xacro:if>
 	<xacro:if value="${not xy_base_joint}">
